Commit message: Multi-myagv control

File: myagv_description/urdf/myAGV.urdf (robot description, URDF)
Before this commit: robot myAGV, 2 links, 1 joints
Links:
- removed link base_footprint
- removed link base_link
- added link ${namespace}base_footprint; visual mesh filename=package://myagv_description/meshes/myagv_base.dae scale=1 1 1
- added link ${namespace}base_link; visual mesh filename=package://myagv_description/meshes/myagv_up.dae scale=1 1 1
- added link ${namespace}camera_link
- added link ${namespace}imu_link
- added link ${namespace}laser_frame
Joints:
- removed joint base_joint
- added joint ${namespace}base_joint: type fixed, parent ${namespace}base_footprint, child ${namespace}base_link, origin xyz=0.0 0.0 0.0 rpy=0 0 0, axis 0 0 1
- added joint ${namespace}base_to_camera: type fixed, parent ${namespace}base_footprint, child ${namespace}camera_link, origin xyz=0.13 0 0.131 rpy=0 0 0
- added joint ${namespace}base_to_imu: type fixed, parent ${namespace}base_footprint, child ${namespace}imu_link, origin xyz=0 0 0 rpy=0 3.14159 3.14159
- added joint ${namespace}base_to_laser: type fixed, parent ${namespace}base_footprint, child ${namespace}laser_frame, origin xyz=0.065 0.0 0.08 rpy=3.14159265 0.0 0.0
